Commit message: feat: add collision and ros2_control, disable self-collision

File: ros2_ws/src/my_robot_description/urdf/assemply.urdf (robot description, URDF)
Before this commit: robot my_robot, 5 links, 4 joints
Links:
- link base_link: geometry collision mesh filename=package://my_robot_description/meshes/base_link_collision.s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; visual mesh filename=package://my_robot_description/meshes/base_link_visual.obj
- link left_wheel: geometry collision mesh filename=package://my_robot_description/meshes/left_wheel_collision.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; visual mesh filename=package://my_robot_description/meshes/left_wheel_visual.obj
- link pan_face: geometry collision mesh filename=package://my_robot_description/meshes/pan_face_collision.stl; visual mesh filename=package://my_robot_description/meshes/pan_face_visual.obj
- link right_wheel: geometry collision mesh filename=package://my_robot_description/meshes/right_wheel_collision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; visual mesh filename=package://my_robot_description/meshes/right_wheel_visual.obj
- link tilt_body: geometry collision mesh filename=package://my_robot_description/meshes/tilt_body_collision.s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; visual mesh filename=package://my_robot_description/meshes/tilt_body_visual.obj

Commit message: fix: clean up URDF TF frames (align link frames with base_link)

File: ros2_ws/src/my_robot_description/urdf/assemply.urdf (robot description, URDF)
Before this commit: robot my_robot, 5 links, 4 joints
Joints:
- joint left_wheel_joint: axis -1 0 0 -> 0 1 0; limit lower=0 upper=0 effort=10 velocity=1 -> effort=10 velocity=1; origin xyz=-0.004905 0.0422 0.05257 rpy=0 0 -1.570796 -> xyz=-0.004905 0.0422 0.05257 rpy=0 0 0
- joint pan_face_joint: axis 0 0 1 -> -1 0 0; limit lower=0 upper=0 effort=10 velocity=1 -> effort=10 velocity=1; origin xyz=-0.05275 -1.851588e-09 1.863159e-08 rpy=-1.570797 -8.742277e-08 -1.570796 -> xyz=0.05275 0 0 rpy=0 0 0
- joint right_wheel_joint: axis 0 0 1 -> 0 1 0; limit lower=0 upper=0 effort=10 velocity=1 -> effort=10 velocity=1; origin xyz=-0.004905 -0.0472 0.05257 rpy=-1.570796 -1.570796 0 -> xyz=-0.004905 -0.0472 0.05257 rpy=0 0 0
- joint tilt_body_joint: origin xyz=-0.004905 -1.916532e-09 0.05257 rpy=8.742278e-08 3.141592 3.178652e-08 -> xyz=-0.004905 0 0.05257 rpy=0 0 0

Commit message: fix: compute link inertia from meshes (nylon PA12)

File: ros2_ws/src/my_robot_description/urdf/assemply.urdf (robot description, URDF)
Before this commit: robot my_robot, 5 links, 4 joints
Links:
- link base_link: mass 0.188891 -> 0.141348
- link left_wheel: mass 0.056299 -> 0.051660
- link pan_face: mass 0.038477 -> 0.037477
- link right_wheel: mass 0.056299 -> 0.051660
- link tilt_body: mass 0.035226 -> 0.028671
