Commit message: feat: add Gazebo Fortress simulation with ros2_control

File: ros2_ws/src/my_robot_description/urdf/my_robot.gazebo.xacro (robot description, xacro)
@@ -1,4 +1,4 @@
 <?xml version="1.0"?>
-<!-- Gazebo-only settings -->
+<!-- Gazebo (Fortress) settings -->
 <robot xmlns:xacro="http://www.ros.org/wiki/xacro">
   <!-- Disable collisions between this robot's own links. External collisions remain enabled. -->
@@ -9,10 +9,18 @@
   </xacro:macro>
   <xacro:no_self_collide link="base_link" />
-  <xacro:no_self_collide link="left_wheel" />
-  <xacro:no_self_collide link="right_wheel" />
   <xacro:no_self_collide link="tilt_body" />
   <xacro:no_self_collide link="pan_face" />
+  <!-- Wheels: grippy rubber-like contact so they roll instead of slide -->
+  <xacro:macro name="wheel_contact" params="link">
+    <gazebo reference="${link}">
+      <selfCollide>false</selfCollide>
+      <mu1>1.0</mu1>
+      <mu2>1.0</mu2>
+    </gazebo>
+  </xacro:macro>
+  <xacro:wheel_contact link="left_wheel" />
+  <xacro:wheel_contact link="right_wheel" />
   <gazebo>
-    <plugin name="gazebo_ros2_control" filename="gz_ros2_control::GazeboSimROS2ControlPlugin">
+    <plugin filename="libgz_ros2_control-system.so" name="gz_ros2_control::GazeboSimROS2ControlPlugin">
       <parameters>$(find my_robot_description)/config/controllers.yaml</parameters>
     </plugin>

File: ros2_ws/src/my_robot_description/urdf/my_robot.urdf.xacro (robot description, xacro)
@@ -1,5 +1,5 @@
 <?xml version="1.0"?>
 <!--
-  my_robot: two-wheeled base with a tilt body and a pan face.
+  my_robot - two-wheeled base with a tilt body and a pan face.
   Build the plain URDF with:
     xacro my_robot.urdf.xacro > my_robot.urdf

File: ros2_ws/src/my_robot_description/urdf/my_robot_core.xacro (robot description, xacro)
@@ -64,5 +64,5 @@
   <xacro:wheel side="right" y="${right_wheel_y}"
     mesh_xyz="0 0.00075 0" mesh_rpy="${-half_pi} ${-half_pi} 0" />
-  <!-- Tilt body: pitches about the wheel axle -->
+  <!-- Tilt body, pitches about the wheel axle -->
   <link name="tilt_body">
     <xacro:tilt_body_inertial />
@@ -78,5 +78,5 @@
     <limit effort="${effort_limit}" velocity="${velocity_limit}" lower="${-pi}" upper="${pi}" />
   </joint>
-  <!-- Pan face: spins about the forward axis at the front of the tilt body -->
+  <!-- Pan face, spins about the forward axis at the front of the tilt body -->
   <link name="pan_face">
     <xacro:pan_face_inertial />

Commit message: feat: multi-module simulation with namespaces and ground-truth pose

File: ros2_ws/src/my_robot_description/urdf/my_robot.gazebo.xacro (robot description, xacro)
@@ -22,6 +22,21 @@
   <xacro:wheel_contact link="right_wheel" />
   <gazebo>
+    <!-- One controller_manager per module, inside the module's namespace -->
     <plugin filename="libgz_ros2_control-system.so" name="gz_ros2_control::GazeboSimROS2ControlPlugin">
       <parameters>$(find my_robot_description)/config/controllers.yaml</parameters>
+      <ros>
+        <namespace>/${namespace}</namespace>
+      </ros>
+    </plugin>
+    <!--
+      Ground-truth pose ("known exact location") straight from the physics engine,
+      published as Gazebo odometry and as TF world -> <prefix>base_link.
+      The launch file bridges both to ROS.
+    -->
+    <plugin filename="ignition-gazebo-odometry-publisher-system" name="ignition::gazebo::systems::OdometryPublisher">
+      <odom_frame>world</odom_frame>
+      <robot_base_frame>${frame_prefix}base_link</robot_base_frame>
+      <dimensions>3</dimensions>
+      <odom_publish_frequency>50</odom_publish_frequency>
     </plugin>
   </gazebo>

File: ros2_ws/src/my_robot_description/urdf/my_robot.urdf.xacro (robot description, xacro)
@@ -4,6 +4,12 @@
   Build the plain URDF with:
     xacro my_robot.urdf.xacro > my_robot.urdf
+  For one module of many in simulation:
+    xacro my_robot.urdf.xacro namespace:=module_1
 -->
 <robot name="my_robot" xmlns:xacro="http://www.ros.org/wiki/xacro">
+  <!-- ROS namespace of this module, e.g. module_1. Empty for a single robot. -->
+  <xacro:arg name="namespace" default="" />
+  <xacro:property name="namespace" value="$(arg namespace)" />
+  <xacro:property name="frame_prefix" value="${namespace + '/' if namespace else ''}" />
   <xacro:include filename="$(find my_robot_description)/urdf/inertial.xacro" />
   <xacro:include filename="$(find my_robot_description)/urdf/my_robot_core.xacro" />
